File: line-in.kicad_sch (KiCad schematic)
At the start: 7 parts

Commit message: More schematic tidying
Other:
- moved on the sheet: C53, C56, C58, L2, L3, MOV1
Changed lines of the file:
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@@
-	)
-	(junction
-		(at 114.3 58.42)
-		(diameter 0)
-		(color 0 0 0 0)
 	)
 	(junction
@@
 	(wire
 		(pts
+			(xy 111.76 49.53) (xy 114.3 49.53)
+		)
+		(stroke
+			(width 0)
+			(type default)
+		)
+	)
+	(wire
+		(pts
 			(xy 130.81 72.39) (xy 130.81 82.55)
 		)
@@
 	(wire
 		(pts
-			(xy 111.76 63.5) (xy 134.62 63.5)
-		)
-		(stroke
-			(width 0)
-			(type default)
-		)
-	)
-	(wire
-		(pts
 			(xy 130.81 90.17) (xy 130.81 96.52)
 		)
@@
 	(wire
 		(pts
-			(xy 111.76 63.5) (xy 111.76 72.39)
-		)
-		(stroke
-			(width 0)
-			(type default)
-		)
-	)
-	(wire
-		(pts
-			(xy 130.81 58.42) (xy 130.81 72.39)
-		)
-		(stroke
-			(width 0)
-			(type default)
-		)
-	)
-	(wire
-		(pts
-			(xy 111.76 58.42) (xy 114.3 58.42)
-		)
-		(stroke
-			(width 0)
-			(type default)
-		)
-	)
-	(wire
-		(pts
 			(xy 130.81 72.39) (xy 133.35 72.39)
 		)
@@
 	(wire
 		(pts
-			(xy 134.62 41.91) (xy 129.54 41.91)
-		)
-		(stroke
-			(width 0)
-			(type default)
-		)
-	)
-	(wire
-		(pts
-			(xy 114.3 58.42) (xy 114.3 49.53)
+			(xy 130.81 41.91) (xy 129.54 41.91)
+		)
+		(stroke
+			(width 0)
+			(type default)
+		)
+	)
+	(wire
+		(pts
+			(xy 111.76 49.53) (xy 111.76 72.39)
 		)
 		(stroke
@@
 	(wire
 		(pts
+			(xy 130.81 41.91) (xy 130.81 72.39)
+		)
+		(stroke
+			(width 0)
+			(type default)
+		)
+	)
+	(wire
+		(pts
 			(xy 124.46 72.39) (xy 130.81 72.39)
 		)
@@
 		(pts
 			(xy 106.68 72.39) (xy 111.76 72.39)
-		)
-		(stroke
-			(width 0)
-			(type default)
-		)
-	)
-	(wire
-		(pts
-			(xy 114.3 58.42) (xy 130.81 58.42)
-		)
-		(stroke
-			(width 0)
-			(type default)
-		)
-	)
-	(wire
-		(pts
-			(xy 134.62 41.91) (xy 134.62 63.5)
 		)
 		(stroke
@@
 	(hierarchical_label "NEUTRAL_IN"
 		(shape passive)
-		(at 111.76 106.68 270)
+		(at 130.81 106.68 270)
 		(effects
 			(font
@@
 	(hierarchical_label "LIVE_IN"
 		(shape passive)
-		(at 130.81 106.68 270)
+		(at 111.76 106.68 270)
 		(effects
 			(font
@@
 	(hierarchical_label "NEUTRAL_SENSE"
 		(shape passive)
-		(at 111.76 63.5 180)
+		(at 130.81 58.42 0)
 		(effects
 			(font
 				(size 1.27 1.27)
 			)
-			(justify right)
+			(justify left)
 		)
 	)
@@
 	(symbol
 		(lib_id "Device:C")
-		(at 102.87 72.39 90)
+		(at 137.16 72.39 270)
 		(unit 1)
 		(exclude_from_sim no)
@@
 		(fields_autoplaced yes)
 		(property "Reference" "C58"
-			(at 102.87 64.77 90)
+			(at 137.16 64.77 90)
 			(effects
 				(font
@@
 		)
 		(property "Value" "4.7nF"
-			(at 102.87 67.31 90)
+			(at 137.16 67.31 90)
 			(effects
 				(font
@@
 		)
 		(property "Footprint" "Capacitor_THT:C_Disc_D10.0mm_W2.5mm_P5.00mm"
-			(at 106.68 71.4248 0)
+			(at 133.35 73.3552 0)
 			(effects
 				(font
@@
 		)
 		(property "Datasheet" "~"
-			(at 102.87 72.39 0)
+			(at 137.16 72.39 0)
 			(effects
 				(font
@@
 		)
 		(property "Description" ""
-			(at 102.87 72.39 0)
+			(at 137.16 72.39 0)
 			(effects
 				(font
@@
 	(symbol
 		(lib_id "Device:C")
-		(at 137.16 72.39 90)
+		(at 102.87 72.39 270)
 		(unit 1)
 		(exclude_from_sim no)
@@
 		(fields_autoplaced yes)
 		(property "Reference" "C56"
-			(at 137.16 64.77 90)
+			(at 102.87 64.77 90)
 			(effects
 				(font
@@
 		)
 		(property "Value" "4.7nF"
-			(at 137.16 67.31 90)
+			(at 102.87 67.31 90)
 			(effects
 				(font
@@
 		)
 		(property "Footprint" "Capacitor_THT:C_Disc_D10.0mm_W2.5mm_P5.00mm"
-			(at 140.97 71.4248 0)
+			(at 99.06 73.3552 0)
 			(effects
 				(font
@@
 		)
 		(property "Datasheet" "~"
-			(at 137.16 72.39 0)
+			(at 102.87 72.39 0)
 			(effects
 				(font
@@
 		)
 		(property "Description" ""
-			(at 137.16 72.39 0)
+			(at 102.87 72.39 0)
 			(effects
 				(font
@@
 	(symbol
 		(lib_id "Device:L_Ferrite")
-		(at 130.81 86.36 0)
+		(at 111.76 86.36 0)
 		(unit 1)
 		(exclude_from_sim no)
@@
 		(fields_autoplaced yes)
 		(property "Reference" "L3"
-			(at 133.35 85.0899 0)
+			(at 114.3 85.0899 0)
 			(effects
 				(font
@@
 		)
 		(property "Value" "L_Radial_D14.2mm_P10.00mm_Neosid_SD14"
-			(at 133.35 87.6299 0)
+			(at 114.3 87.6299 0)
 			(effects
 				(font
@@
 		)
 		(property "Footprint" "Inductor_THT:L_Radial_D14.2mm_P10.00mm_Neosid_SD14"
-			(at 130.81 86.36 0)
+			(at 111.76 86.36 0)
 			(effects
 				(font
@@
 		)
 		(property "Datasheet" "~"
-			(at 130.81 86.36 0)
+			(at 111.76 86.36 0)
 			(effects
 				(font
@@
 		)
 		(property "Description" ""
-			(at 130.81 86.36 0)
+			(at 111.76 86.36 0)
 			(effects
 				(font
@@
 	(symbol
 		(lib_id "Device:Varistor")
-		(at 120.65 96.52 90)
+		(at 120.65 96.52 270)
 		(unit 1)
 		(exclude_from_sim no)
@@
 		(fields_autoplaced yes)
 		(property "Reference" "MOV1"
-			(at 120.8433 90.17 90)
+			(at 120.4566 88.9 90)
 			(effects
 				(font
@@
 		)
 		(property "Value" "RV_Disc_D15.5mm_W3.9mm_P7.5mm"
-			(at 120.8433 92.71 90)
+			(at 120.4566 91.44 90)
 			(effects
 				(font
@@
 		)
 		(property "Footprint" "Varistor:RV_Disc_D15.5mm_W3.9mm_P7.5mm"
-			(at 120.65 98.298 90)
+			(at 120.65 94.742 90)
 			(effects
 				(font
@@
 	(symbol
 		(lib_id "Device:L_Ferrite")
-		(at 111.76 86.36 180)
+		(at 130.81 86.36 180)
 		(unit 1)
 		(exclude_from_sim no)
@@
 		(fields_autoplaced yes)
 		(property "Reference" "L2"
-			(at 113.03 85.0899 0)
+			(at 132.08 85.0899 0)
 			(effects
 				(font
@@
 		)
 		(property "Value" "L_Radial_D14.2mm_P10.00mm_Neosid_SD14"
-			(at 113.03 87.6299 0)
+			(at 132.08 87.6299 0)
 			(effects
 				(font
@@
 		)
 		(property "Footprint" "Inductor_THT:L_Radial_D14.2mm_P10.00mm_Neosid_SD14"
-			(at 111.76 86.36 0)
+			(at 130.81 86.36 0)
 			(effects
 				(font
@@
 		)
 		(property "Datasheet" "~"
-			(at 111.76 86.36 0)
+			(at 130.81 86.36 0)
 			(effects
 				(font
@@
 		)
 		(property "Description" ""
-			(at 111.76 86.36 0)
+			(at 130.81 86.36 0)
 			(effects
 				(font
@@
 	(symbol
 		(lib_id "Device:C")
-		(at 120.65 72.39 270)
+		(at 120.65 72.39 90)
 		(unit 1)
 		(exclude_from_sim no)
@@
 		)
 		(property "Footprint" "apc-custom:C_Rect_L31.5mm_W13.0mm_P27.50mm_MKS4_Doublesided"
-			(at 116.84 73.3552 0)
-			(effects
-				(font
+			(at 124.46 71.4248 0)
+			(effects
+				(font
