File: pcb.kicad_sch (KiCad schematic)
At the start: 241 parts, among them J17 PinHeader_1x04_P7.00mm_Vertic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, Q1 TO-92_Inline_Wide_Doublesided, Q10 TO-92_Inline_Wide_Doublesided, Q11 TO-92_Inline_Wide_Doublesided, Q12 TO-220F-3_Vertical_Doublesided, Q13 TO-220F-3_Vertical_Doublesided, Q14 TO-220F-3_Vertical_Doublesided, Q15 TO-220F-3_Vertical_Doublesided, Q18 TO-220F-3_Vertical_Doublesided, Q19 TO-220F-3_Vertical_Doublesided, Q2 TO-92_Inline_Wide_Doublesided, Q23 TO-92_Inline_Wide_Doublesided, Q24 TO-92_Inline_Wide_Doublesided, Q25 TO-92_Inline_Wide_Doublesided, Q26 TO-92_Inline_Wide_Doublesided, Q27 TO-92_Inline_Wide_Doublesided, Q28 TO-92_Inline_Wide_Doublesided, Q3 TO-92_Inline_Wide_Doublesided, Q4 TO-92_Inline_Wide_Doublesided, Q5 TO-92_Inline_Wide_Doublesided, Q6 TO-92_Inline_Wide_Doublesided, Q7 TO-92_Inline_Wide_Doublesided, Q8 TO-92_Inline_Wide_Doublesided, Q9 MPSA43, T1 Transformer_T1, U1 DIP-40_W15.24mm_Socket, U2 DIP-24_W7.62mm, U3 DIP-8_W7.62mm, U5 TO-92_Inline_Wide_Doublesided, U6 DIP-14_W7.62mm_Doublesided, U7 DIP-6_W7.62mm, U8 TO-220F-5_P3.4x3.7mm_StaggerE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, U9 DIP-14_W7.62mm_Doublesided, Y1 Crystal_HC52-U_Vertical

Commit message: More schematic tidying
Parts:
- added T3: Transformer_SC420, symbol apc-custom:Transformer_SC420
- BP1: value MagneticBuzzer_ProSignal_ABT-410-RC -> 390-0004
- BT1: value Battery -> 12V
- C10: value C_Tant_L9.0mm_W2.5mm_P7.50mm_MKT -> 10nF
- C13, C14: value C_Disc_D4.7mm_W2.5mm_P5.00mm_Doublesided -> 22pF
- C15, C42: value C_Radial_D12.5mm_H25.0mm_P5.00mm_Doublesided -> 1000uF 50V
- C21, C22, C60: value C_Tant_L9.0mm_W2.5mm_P7.50mm_MKT -> 100nF
- C24, C68: value C_Tant_L5.0mm_W2.5mm_P5.0mm_MKT_Doublesided -> 1uF
- C25, C29, C33, C34, C43, C45, C47, C48, C51: value C_Rect_L7.0mm_W2.0mm_P5.00mm_Doublesided -> .1uF 63V
- C27, C28, C36, C37: value C_Rect_L7.0mm_W2.0mm_P5.00mm_Doublesided -> 22nF 100V
- C30, C31, C35, C38, C49, C50: value C_Radial_D4.0mm_H7.0mm_P5.00mm_Doublesided -> 22uF 16V
- C32: value C_Disc_D4.7mm_W2.5mm_P5.00mm_Doublesided -> 470pF
- C39, C61: value C_Rect_L7.0mm_W2.0mm_P5.00mm_Doublesided -> 4.7nF 63V
- C40: value R_Axial_DIN0207_L6.3mm_D2.5mm_P10.16mm_Horizontal_Doublesided -> .22uF 63V
- C46: footprint (none) -> apc-custom:C_Rect_L7.0mm_W2.0mm_P5.00mm_Doublesided
- C5: value 100nF -> 1uF
- C55: value C_Rect_L18.0mm_W5.0mm_P15.00mm_FKS3_FKP3_Doublesided -> 22uF 275V
- D44: symbol Device:D_Zener -> Device:D
- Q1, Q24, Q25: value TO-92_Inline_Wide_Doublesided -> MPSA13
- Q10, Q27, Q3, Q5, Q7: value TO-92_Inline_Wide_Doublesided -> KSP2222A
- Q11, Q2, Q26, Q4, Q6: value TO-92_Inline_Wide_Doublesided -> KSP2907A
- Q12, Q13: value TO-220F-3_Vertical_Doublesided -> IRFZ34N
- Q23, Q28, Q8: value TO-92_Inline_Wide_Doublesided -> 2N7000
- R1, R19, R42, R43: value R_Axial_DIN0207_L6.3mm_D2.5mm_P10.16mm_Horizontal_Doublesided -> 47K
- R100, R107, R17, R21, R38, R63, R69, R70, R71, R8, R9, R90, R91, R98: value R_Axial_DIN0207_L6.3mm_D2.5mm_P10.16mm_Horizontal_Doublesided -> 10K
- R105, R23, R24, R29, R30, R37, R64, R99: value R_Axial_DIN0207_L6.3mm_D2.5mm_P10.16mm_Horizontal_Doublesided -> 1K
- R108, R13, R20, R34, R36, R44, R72, R82: value R_Axial_DIN0207_L6.3mm_D2.5mm_P10.16mm_Horizontal_Doublesided -> 20K
- R12, R16: value R_Axial_DIN0207_L6.3mm_D2.5mm_P10.16mm_Horizontal_Doublesided -> 4.7K
- R18, R2, R22: value R_Axial_DIN0207_L6.3mm_D2.5mm_P10.16mm_Horizontal_Doublesided -> 47R
- R26, R33: value R_Axial_DIN0207_L6.3mm_D2.5mm_P10.16mm_Horizontal_Doublesided -> 10K7
- R3: value R_Axial_DIN0207_L6.3mm_D2.5mm_P10.16mm_Horizontal_Doublesided -> 887K
- R39, R40, R41: value R_Axial_DIN0411_L9.9mm_D3.6mm_P15.24mm_Horizontal -> 39K
- R4: value R_Axial_DIN0207_L6.3mm_D2.5mm_P10.16mm_Horizontal_Doublesided -> 470R
- R5: value R_Axial_DIN0207_L6.3mm_D2.5mm_P10.16mm_Horizontal_Doublesided -> 330R
- R52, R57: value R_Axial_DIN0207_L6.3mm_D2.5mm_P10.16mm_Horizontal_Doublesided -> 10K3
- R6, R7: value R_Axial_DIN0207_L6.3mm_D2.5mm_P10.16mm_Horizontal_Doublesided -> 680R
- R65: value R_Axial_DIN0516_L15.5mm_D5.0mm_P20.32mm_Horizontal_Doublesided -> 0.59R
- R92: value R_Axial_DIN0207_L6.3mm_D2.5mm_P10.16mm_Horizontal_Doublesided -> ~
- RLY2, RLY4: value Relay_SPDT_Schrack-RT1-FormC_RM3.5mm -> O/E/N 450-0026 59-12-1CE
- RLY3: value Relay_SPDT_Schrack-RT1-FormC_RM3.5mm -> JW1FSN-B-DC12V
- T1: value Transformer_T1 -> 460-0008-2
- U2: value DIP-24_W7.62mm -> JH418AE
- U5: value TO-92_Inline_Wide_Doublesided -> MSC34064
- U6: value DIP-14_W7.62mm_Doublesided -> LM324AN
- U7: value DIP-6_W7.62mm -> 4N25-X001
- U9: value DIP-14_W7.62mm_Doublesided -> UEYW0418
- VR1: value TO-92_Inline_Wide_Doublesided -> 2950
- Y1: value Crystal_HC52-U_Vertical -> CREC 16MHz
Connections:
- net Line in/RLY_LINE_2 is gone; now on net PLUS_12V: C52.2, F1.2, Q2.1 (C), Q6.1 (C), R36.2, RLY2.A2, RLY3.A1, RLY4.A2, U7.5
- net Front Panel/FP_PWR: now also R17.2; no longer R17.1
- net GND: now also D44.2 (A), Q23.1 (S), Q24.1 (C), R90.2, U1.20 (VSS); no longer U3.5 (GND)
- net TX_BLU: now also T3.6 (SB)
- net TX_BRN: now also T3.5 (SA)
- net TX_WHT: now also T3.4 (AD)
- net at C15.1, C42.1, C43.1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: no longer C39.1
- net RLY2_CTRL: now reaches Q24.2 (B), R96.1
- net RLY2_ACT: now reaches D39.2 (A), Q24.3 (E), RLY2.A1
- net at D44.1 (K), Q23.2 (G): no longer R90.2
- net at C23.1, R12.1, R13.1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: now also U2.6 (CH5)
- net at Q11.2 (B), R64.1: now also C39.1
- net at BP1.1 (+), C8.1, D42.2 (A)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: now also R17.1
- net at C8.2, Q2.2 (B), R16.2: no longer R17.2
- net at Q12.1 (G), Q13.1 (G): now also R63.1, R68.1
- net at C6.2, R3.2, R8.1: now also U2.9 (CH8)
- net RLY3_ACT: now reaches D35.2 (A), Q25.3 (E), RLY3.A2
- net at C62.1, C68.2, L4.1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: now also U2.11 (VREF)
- net at D14.2 (A), D15.1 (K), R56.2: now also U2.5 (CH4)
- net at Q5.3 (C): now also U1.12 (P3.2/~{INT0})
- net PLUS_12V: now reaches Q27.2 (B), R100.1, R99.1
- net PLUS_12V: now also D38.2 (A)
- net CHARGE_CTRL: now reaches R107.1, U8.5 (~{ON}/OFF)
- net at U1.16 (P3.6/~{WR}), U3.4 (DO): no longer R107.2
- net RLY4_ACT: now reaches D36.2 (A), Q27.3 (C), RLY4.A1
- net at U2.1 (~{RD}): now also U1.1 (P1.0/T2)
- net ADC-D7: now reaches U2.13 (DB7)
- net ADC-D7: now also U1.28 (P2.7/A15)
- net ADC-D6: now reaches U2.14 (DB6)
- net ADC-D6: now also U1.27 (P2.6/A14)
- net ADC-D5: now reaches U2.15 (DB5)
- net ADC-D5: now also U1.26 (P2.5/A13)
- net ADC-D4: now reaches U2.16 (DB4/MA4)
- net ADC-D4: now also U1.25 (P2.4/A12)
- net ADC-D3: now reaches U2.17 (DM3/MA3)
- net ADC-D3: now also U1.24 (P2.3/A11)
- net ADC-D2: now reaches U2.18 (DB2/MA2)
- net ADC-D2: now also U1.23 (P2.2/A10)
- net ADC-D1: now reaches U2.19 (DB1/MA1)
- net ADC-D1: now also U1.22 (P2.1/A9)
- net ADC-D0: now reaches U2.20 (DB0/MA0)
- net ADC-D0: now also U1.21 (P2.0/A8)
- net at U2.22 (~{WR}): now also U1.2 (P1.1/T2EX)
- net at U2.23 (~{CS}): now also U1.3 (P1.2/ECI)
- net RLY3_CTRL: now reaches Q25.2 (B), R97.1
- net at U1.17 (P3.7/~{RD}): now also R107.2
- net at U1.6 (P1.5/CEX2): now also R90.1
- net at U1.7 (P1.6/CEX3): now also R96.2
- net at U1.8 (P1.7/CEX4): now also R97.2
- net Line in/RLY_LINE_1 renamed RLY1_ACT
Other:
- moved on the sheet: C10, C11, C12, C15, C21, C22, C24, C25, C27, C39, C40, C41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

Commit message: Add placeholder components for unknown ICs
Finish the serial interface schematic
Parts:
- removed C21, C22: 100nF, apc-custom:C_Tant_L9.0mm_W2.5mm_P7.50mm_MKT, symbol Device:C
- removed U9: UEYW0418, apc-custom:DIP-14_W7.62mm_Doublesided, symbol apc-custom:360-2040B
- added U9: Conn_02x07_Counter_Clockwise, apc-custom:DIP-14_W7.62mm_Doublesided, symbol Connector_Generic:Conn_02x07_Counter_Clockwise
Connections:
- net GND: now also U9.5 (Pin_5)
- net at R70.2: now also U9.8 (Pin_8)
- net at R73.1, R82.2, R83.2: now also U9.12 (Pin_12)
- net at R72.1, R78.2, R79.2: now also U9.10 (Pin_10)
- net at C46.2: now also U9.2 (Pin_2)
- net at C49.1, R1.1, R75.1: now also U9.14 (Pin_14)
- net at C48.1, R75.2: now also U9.13 (Pin_13)
- net at C45.1, D26.1 (K), D46.1 (K)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: now also U9.7 (Pin_7)
- net Serial interface/VCC: now reaches C57.1, Q6.3 (E), R46.1, U6.4 (V+)
- net Serial interface/VCC: now also U9.1 (Pin_1)
- net at R71.2: now also U9.9 (Pin_9)
- net Serial interface/TxD: now reaches R91.1
- net at C47.2: now also U9.4 (Pin_4)
- net at R76.1, R77.1: now also U9.6 (Pin_6)
- net Serial interface/PIN12: now reaches R13.2
- net at R68.2: now also U9.11 (Pin_11)
- net Serial interface/RxD: now reaches R106.1
- net Serial interface/PIN11: now reaches R12.2
- net at R74.1: now also U9.3 (Pin_3)
- net Serial interface/PIN10: now reaches U1.35 (P0.4/AD4)
- no-connect marks 0 -> 1
Other:
- sheet Serial interface ports: added PIN10, PIN11, PIN12, RxD, TxD, VCC; removed none
- moved on the sheet: C24, Q3, R12, R13, R18, R19, R20, R70, R71

Commit message: Fix a few misconnected wires
Connections:
- net Front Panel/FP_PWR: now also R17.1; no longer R17.2
- net GND: no longer R90.2
- net PLUS_12V: no longer Q27.2 (B), R100.1, R99.1
- net RLY1_CTRL: now reaches D44.1 (K), Q23.2 (G)
- net RLY1_CTRL: now also R90.2
- net at BP1.1 (+), C8.1, D42.2 (A)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: no longer R17.1
- net at C8.2, Q2.2 (B), R16.2: now also R17.2
- net at C27.1, D9.1 (K), R26.2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: now also C27.2, R26.1, R28.1, U6.2 (-)
- new net RLY4_CTRL: Q27.2 (B), R100.1, R99.1
Other:
- moved on the sheet: C27, C28, C37, C46, C47, C48, C51, D27, D32, D44, Q11, R17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

Commit message: More schematic tidyups
Connections:
- net at R86.1: now also D30.1 (K), D31.1 (K), R88.2
Other:
- moved on the sheet: R75, R86, R87

Commit message: Populate some more resistor values, add some missing wires
Parts:
- R106, R56: value R_Axial_DIN0207_L6.3mm_D2.5mm_P10.16mm_Horizontal_Doublesided -> 1K
- R45: value R_Axial_DIN0207_L6.3mm_D2.5mm_P10.16mm_Horizontal_Doublesided -> 2M
- R46, R77, R86: value R_Axial_DIN0207_L6.3mm_D2.5mm_P10.16mm_Horizontal_Doublesided -> 10K
- R47: value R_Axial_DIN0207_L6.3mm_D2.5mm_P10.16mm_Horizontal_Doublesided -> 200R
- R58: value R_Axial_DIN0207_L6.3mm_D2.5mm_P10.16mm_Horizontal_Doublesided -> 4K02 1%
- R59: value R_Axial_DIN0207_L6.3mm_D2.5mm_P10.16mm_Horizontal_Doublesided -> 3K12 1%
- R61: value R_Axial_DIN0207_L6.3mm_D2.5mm_P10.16mm_Horizontal_Doublesided -> 10K 1%
- R62: value R_Axial_DIN0207_L6.3mm_D2.5mm_P10.16mm_Horizontal_Doublesided -> 1K 1%
- R66: value R_Axial_DIN0207_L6.3mm_D2.5mm_P10.16mm_Horizontal_Doublesided -> 26.4K 0.1%
- R67: value R_Axial_DIN0207_L6.3mm_D2.5mm_P10.16mm_Horizontal_Doublesided -> 2.43K 0.1%
- R68: value R_Axial_DIN0207_L6.3mm_D2.5mm_P10.16mm_Horizontal_Doublesided -> 100R
- R73: value R_Axial_DIN0207_L6.3mm_D2.5mm_P10.16mm_Horizontal_Doublesided -> 20K
- R74: value R_Axial_DIN0207_L6.3mm_D2.5mm_P10.16mm_Horizontal_Doublesided -> 200K 1%
- R75: value R_Axial_DIN0207_L6.3mm_D2.5mm_P10.16mm_Horizontal_Doublesided -> 3K01 1%
- R78, R79, R83: value R_Axial_DIN0207_L6.3mm_D2.5mm_P10.16mm_Horizontal_Doublesided -> 47R
- R87: value R_Axial_DIN0207_L6.3mm_D2.5mm_P10.16mm_Horizontal_Doublesided -> 604K 1%
- R88: value R_Axial_DIN0207_L6.3mm_D2.5mm_P10.16mm_Horizontal_Doublesided -> 2K 1%
- R89: value R_Axial_DIN0207_L6.3mm_D2.5mm_P10.16mm_Horizontal_Doublesided -> 1.5K 1%
- R92: value ~ -> 1.5K 1%
- R95: value R_Axial_DIN0207_L6.3mm_D2.5mm_P10.16mm_Horizontal_Doublesided -> 680K
- R96, R97: value R_Axial_DIN0207_L6.3mm_D2.5mm_P10.16mm_Horizontal_Doublesided -> 100K
Connections:
- net GND: now also C5.1, Q28.1 (S), U3.5 (GND)
- net at Q28.3 (D), R86.2, R87.2: now also C51.2
- net at R1.2, R108.2: now also U1.34 (P0.5/AD5)
- net at R87.1, U2.7 (CH6): no longer C51.2
- no-connect marks 1 -> 4
Other:
- moved on the sheet: C51, D44, D45, R3, R71, R73, R82, R86, R87
