File: pcb.kicad_sch (KiCad schematic)
At the start: 240 parts, among them J17 PinHeader_1x04_P7.00mm_Vertic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, Q1 MPSA13, Q10 KSP2222A, Q11 KSP2907A, Q12 IRFZ34N, Q13 IRFZ34N, Q14 TO-220F-3_Vertical_Doublesided, Q15 TO-220F-3_Vertical_Doublesided, Q18 TO-220F-3_Vertical_Doublesided, Q19 TO-220F-3_Vertical_Doublesided, Q2 KSP2907A, Q23 2N7000, Q24 MPSA13, Q25 MPSA13, Q26 KSP2907A, Q27 KSP2222A, Q28 2N7000, Q3 KSP2222A, Q4 KSP2907A, Q5 KSP2222A, Q6 KSP2907A, Q7 KSP2222A, Q8 2N7000, Q9 MPSA43, T1 460-0008-2, T3 Transformer_SC420, U1 DIP-40_W15.24mm_Socket, U2 JH418AE, U3 DIP-8_W7.62mm, U5 MSC34064, U6 LM324AN, U7 4N25-X001, U8 TO-220F-5_P3.4x3.7mm_StaggerE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, U9 Conn_02x07_Counter_Clockwise, Y1 CREC 16MHz

Commit message: Clean up the power network
Parts:
- C5: footprint apc-custom:C_Tant_L9.0mm_W2.5mm_P7.50mm_MKT -> apc-custom:C_Tant_L5.0mm_W2.5mm_P5.0mm_MKT_Doublesided
Connections:
- net VCC: no longer L4.2, L5.2, R2.1, R70.1, R71.1, R9.2
- net OUT_SENSE: now reaches D30.1 (K), D31.1 (K), R86.1, R88.2
- net at Q28.3 (D), R86.2, R87.2: no longer C51.2
- net at C27.1, D9.1 (K), R26.2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: no longer C27.2, R26.1, R28.1, U6.2 (-)
- net at R87.1, U2.7 (CH6): now also C51.2
- net OVLD: now reaches C11.1, R5.2, U1.38 (P0.1/AD1)
- net LINE_IN_SW: now reaches R90.1, U1.6 (P1.5/CEX2)
- new net: L4.2, L5.2, R2.1, R70.1, R71.1, R9.2
- new net: C27.2, R26.1, R28.1, U6.2 (-)
Other:
- moved on the sheet: C51, C52, C7, L4, R16
