File: pcb.kicad_sch (KiCad schematic)
At the start: 240 parts, among them J17 PinHeader_1x04_P7.00mm_Vertic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, Q1 MPSA13, Q10 KSP2222A, Q11 KSP2907A, Q12 IRFZ34N, Q13 IRFZ34N, Q14 TO-220F-3_Vertical_Doublesided, Q15 TO-220F-3_Vertical_Doublesided, Q18 TO-220F-3_Vertical_Doublesided, Q19 TO-220F-3_Vertical_Doublesided, Q2 KSP2907A, Q23 2N7000, Q24 MPSA13, Q25 MPSA13, Q26 KSP2907A, Q27 KSP2222A, Q28 2N7000, Q3 KSP2222A, Q4 KSP2907A, Q5 KSP2222A, Q6 KSP2907A, Q7 KSP2222A, Q8 2N7000, Q9 MPSA43, T1 460-0008-2, T3 Transformer_SC420, U1 DIP-40_W15.24mm_Socket, U2 JH418AE, U3 DIP-8_W7.62mm, U5 MSC34064, U6 LM324AN, U7 4N25-X001, U8 TO-220F-5_P3.4x3.7mm_StaggerE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, U9 Conn_02x07_Counter_Clockwise, Y1 CREC 16MHz

Commit message: Clean up the inverter schematic
It's now a lot clearer how the inverter is laid out, with the centre tap
on the transformer linking to the battery positive, and the two taps
either side being alternately connected to ground, generating a square
wave through the transformer.

There are 3 control/sense lines connecting to mystery IC U9
Parts:
- D13: value D_DO-34_SOD68_P10.16mm_Horizontal_Doublesided -> 1N4148
- J10, J11, J12, J13, J15, J16, J4, J5, J6, J7, J8: value ~ -> (none)
Connections:
- net OUTWHT: now also T3.1 (AA)
- net TX_BLK: now also T3.8 (SD)
- net TX_RED: now also T3.9 (SE)
- net TX_WHT: now also T3.7 (SC); no longer T3.4 (AD)
- net TX_RED_CTL: now reaches R73.1, R82.2, R83.2, U9.12 (Pin_12)
- net TX_WHT_CTL: now reaches R72.1, R78.2, R79.2, U9.10 (Pin_10)
- net BEEPER_CTL: now reaches R1.2, R108.2, U1.34 (P0.5/AD5)
- net NEUTRAL_D: now reaches J17.3 (Pin_3), RLY3.12
- net NEUTRAL_D: now also T3.3 (AC)
- net NEUTRAL_C: now reaches J17.2 (Pin_2), RLY3.14
- net NEUTRAL_C: now also T3.2 (AB)
- net NEUTRAL_A: now reaches C63.1, J17.4 (Pin_4), RLY2.14
- net NEUTRAL_A: now also T3.4 (AD)
- net LINE_SENSE: now reaches D14.2 (A), D15.1 (K), R56.2, U2.5 (CH4)
- net NEUTRAL_OUT: now reaches R89.2, RLY4.14, T1.3 (SA)
- net RLY3_ACT renamed NEUTRAL_CD_SEL
- net RLY3_CTRL renamed NEUTRAL_CD_CTRL
Other:
- note added: "Battery charge taps"
- note added: "Black"
- note added: "Blue"
- note added: "Brown"
- note added: "Doesn't look right?"
- note added: "Orange"
- note added: "Purple"
- note added: "White"
- note added: "Yellow"
- moved on the sheet: BP1, C23, C29, C30, C45, C46, C47, C5, C55, C67, C8, D25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
